File: PCB/hackpad.kicad_pcb (KiCad board)
At the start: 2 copper layers, 79 x 99 mm, 53 parts, among them J1 Conn_01x04, SW1 SW_Push, SW10 SW_Push, SW11 SW_Push, SW12 SW_Push, SW13 SW_Push, SW14 SW_Push, SW15 SW_Push, SW16 SW_Push, SW2 SW_Push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

Commit message: move kicad libraries to third_party dir, update to kicad 9.0
Parts:
- D17, D18, D19, D20, D21, D22, D23, D24, D25, D26, D27, D28, D29, D30, D31, D32: footprint Keebio-Parts:SK6812-MINI-E -> library_edited:SK6812-MINI-E
- SW1, SW10, SW11, SW12, SW13, SW14, SW15, SW16, SW2, SW3, SW4, SW5, SW6, SW7, SW9: footprint Switch_Keyboard_Kailh:SW_Kailh_Choc_V2_1.00u -> library_edited:SW_Kailh_Choc_V2_1.00u
- SW8: footprint Switch_Keyboard_Kailh:SW_Kailh_Choc_V2_2.00u -> library_edited:SW_Kailh_Choc_V2_1.00u
