File: PCB/hackpad.kicad_sch (KiCad schematic)
At the start: 50 parts, among them J1 Conn_01x04, SW1 SW_Push, SW10 SW_Push, SW11 SW_Push, SW12 SW_Push, SW13 SW_Push, SW14 SW_Push, SW15 SW_Push, SW16 SW_Push, SW2 SW_Push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

Commit message: finalize pcb traces and silkscreen text
Other:
- title: (none) -> colon3pad
Changed lines of the file:
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@@
 	(generator_version "8.0")
 	(paper "A4")
+	(title_block
+		(title "colon3pad")
+		(rev "v1.0")
+	)
 	(junction
 		(at 254 60.96)
@@
 	(label "ROW1"
 		(at 102.87 43.18 0)
+		(fields_autoplaced yes)
 		(effects
 			(font
@@
 	(label "SCL"
 		(at 254 114.3 0)
+		(fields_autoplaced yes)
 		(effects
 			(font
@@
 	(label "COL1"
 		(at 208.28 25.4 0)
+		(fields_autoplaced yes)
 		(effects
 			(font
@@
 	(label "COL4"
 		(at 261.62 25.4 0)
+		(fields_autoplaced yes)
 		(effects
 			(font
@@
 	(label "ROW2"
 		(at 200.66 60.96 0)
+		(fields_autoplaced yes)
 		(effects
 			(font
@@
 	(label "ROW4"
 		(at 102.87 54.61 0)
+		(fields_autoplaced yes)
 		(effects
 			(font
@@
 	(label "DATA"
 		(at 118.11 34.29 0)
+		(fields_autoplaced yes)
 		(effects
 			(font
@@
 	(label "ROW1"
 		(at 200.66 43.18 0)
+		(fields_autoplaced yes)
 		(effects
 			(font
@@
 	(label "COL4"
 		(at 58.42 43.18 0)
+		(fields_autoplaced yes)
 		(effects
 			(font
@@
 	(label "SDA"
 		(at 254 111.76 0)
+		(fields_autoplaced yes)
 		(effects
 			(font
@@
 	(label "SCL"
 		(at 58.42 50.8 0)
+		(fields_autoplaced yes)
 		(effects
 			(font
@@
 	(label "ROW4"
 		(at 200.66 96.52 0)
+		(fields_autoplaced yes)
 		(effects
 			(font
@@
 	(label "COL3"
 		(at 58.42 39.37 0)
+		(fields_autoplaced yes)
 		(effects
 			(font
@@
 	(label "DATA"
 		(at 58.42 54.61 0)
+		(fields_autoplaced yes)
 		(effects
 			(font
@@
 	(label "ROW3"
 		(at 200.66 78.74 0)
+		(fields_autoplaced yes)
 		(effects
 			(font
@@
 	(label "ROW2"
 		(at 102.87 46.99 0)
+		(fields_autoplaced yes)
 		(effects
 			(font
@@
 	(label "COL1"
 		(at 58.42 31.75 0)
+		(fields_autoplaced yes)
 		(effects
 			(font
@@
 	(label "COL2"
 		(at 226.06 25.4 0)
+		(fields_autoplaced yes)
 		(effects
 			(font
@@
 	(label "COL2"
 		(at 58.42 35.56 0)
+		(fields_autoplaced yes)
 		(effects
 			(font
@@
 	(label "SDA"
 		(at 58.42 46.99 0)
+		(fields_autoplaced yes)
 		(effects
 			(font
@@
 	(label "COL3"
 		(at 243.84 25.4 0)
+		(fields_autoplaced yes)
 		(effects
 			(font
@@
 	(label "ROW3"
 		(at 102.87 50.8 0)
-		(effects
-			(font
+		(fields_autoplaced yes)
+		(effects
+			(font

Commit message: move kicad libraries to third_party dir, update to kicad 9.0
Parts:
- U1: footprint OPL:XIAO-RP2040-DIP -> Module:MOUDLE14P-XIAO-DIP-SMD
Changed lines of the file:
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@@
 (kicad_sch
-	(version 20231120)
+	(version 20250114)
 	(generator "eeschema")
-	(generator_version "8.0")
+	(generator_version "9.0")
 	(paper "A4")
 	(title_block
@@
 		(rev "v1.0")
 	)
+	(rectangle
+		(start 115.57 17.78)
+		(end 194.31 115.57)
+		(stroke
+			(width 0)
+			(type default)
+		)
+		(fill
+			(type none)
+		)
+	)
+	(rectangle
+		(start 55.88 17.78)
+		(end 111.76 59.69)
+		(stroke
+			(width 0)
+			(type default)
+		)
+		(fill
+			(type none)
+		)
+	)
+	(rectangle
+		(start 243.84 104.14)
+		(end 280.67 123.19)
+		(stroke
+			(width 0)
+			(type default)
+		)
+		(fill
+			(type none)
+		)
+	)
+	(rectangle
+		(start 198.12 17.78)
+		(end 280.67 100.33)
+		(stroke
+			(width 0)
+			(type default)
+		)
+		(fill
+			(type none)
+		)
+	)
+	(text "OLED Display\n"
+		(exclude_from_sim no)
+		(at 270.002 106.68 0)
+		(effects
+			(font
+				(size 2 2)
+			)
+		)
+	)
+	(text "Neopixel LEDs"
+		(exclude_from_sim no)
+		(at 182.118 20.574 0)
+		(effects
+			(font
+				(size 2 2)
+			)
+		)
+	)
+	(text "Key Matrix"
+		(exclude_from_sim no)
+		(at 271.526 20.32 0)
+		(effects
+			(font
+				(size 2 2)
+			)
+		)
+	)
+	(text "RP2040 MCU\n"
+		(exclude_from_sim no)
+		(at 100.584 20.574 0)
+		(effects
+			(font
+				(size 2 2)
+			)
+		)
+	)
 	(junction
 		(at 254 60.96)
@@
 		)
 	)
-	(rectangle
-		(start 115.57 17.78)
-		(end 194.31 115.57)
-		(stroke
-			(width 0)
-			(type default)
-		)
-		(fill
-			(type none)
-		)
-	)
-	(rectangle
-		(start 55.88 17.78)
-		(end 111.76 59.69)
-		(stroke
-			(width 0)
-			(type default)
-		)
-		(fill
-			(type none)
-		)
-	)
-	(rectangle
-		(start 243.84 104.14)
-		(end 280.67 123.19)
-		(stroke
-			(width 0)
-			(type default)
-		)
-		(fill
-			(type none)
-		)
-	)
-	(rectangle
-		(start 198.12 17.78)
-		(end 280.67 100.33)
-		(stroke
-			(width 0)
-			(type default)
-		)
-		(fill
-			(type none)
-		)
-	)
-	(text "OLED Display\n"
-		(exclude_from_sim no)
-		(at 270.002 106.68 0)
-		(effects
-			(font
-				(size 2 2)
-			)
-		)
-	)
-	(text "Neopixel LEDs"
-		(exclude_from_sim no)
-		(at 182.118 20.574 0)
-		(effects
-			(font
-				(size 2 2)
-			)
-		)
-	)
-	(text "Key Matrix"
-		(exclude_from_sim no)
-		(at 271.526 20.32 0)
-		(effects
-			(font
-				(size 2 2)
-			)
-		)
-	)
-	(text "RP2040 MCU\n"
-		(exclude_from_sim no)
-		(at 100.584 20.574 0)
-		(effects
-			(font
-				(size 2 2)
-			)
-		)
-	)
 	(label "ROW1"
 		(at 102.87 43.18 0)
-		(fields_autoplaced yes)
 		(effects
 			(font
@@
 	(label "SCL"
 		(at 254 114.3 0)
-		(fields_autoplaced yes)
 		(effects
 			(font
@@
 	(label "COL1"
 		(at 208.28 25.4 0)
-		(fields_autoplaced yes)
 		(effects
 			(font
@@
 	(label "COL4"
 		(at 261.62 25.4 0)
-		(fields_autoplaced yes)
 		(effects
 			(font
@@
 	(label "ROW2"
 		(at 200.66 60.96 0)
-		(fields_autoplaced yes)
 		(effects
 			(font
@@
 	(label "ROW4"
 		(at 102.87 54.61 0)
-		(fields_autoplaced yes)
 		(effects
 			(font
@@
 	(label "DATA"
 		(at 118.11 34.29 0)
-		(fields_autoplaced yes)
 		(effects
 			(font
@@
 	(label "ROW1"
 		(at 200.66 43.18 0)
-		(fields_autoplaced yes)
 		(effects
 			(font
@@
 	(label "COL4"
 		(at 58.42 43.18 0)
-		(fields_autoplaced yes)
 		(effects
 			(font
@@
 	(label "SDA"
 		(at 254 111.76 0)
-		(fields_autoplaced yes)
 		(effects
 			(font
@@
 	(label "SCL"
 		(at 58.42 50.8 0)
-		(fields_autoplaced yes)
 		(effects
 			(font
@@
 	(label "ROW4"
 		(at 200.66 96.52 0)
-		(fields_autoplaced yes)
 		(effects
 			(font
@@
 	(label "COL3"
 		(at 58.42 39.37 0)
-		(fields_autoplaced yes)
 		(effects
 			(font
@@
 	(label "DATA"
 		(at 58.42 54.61 0)
-		(fields_autoplaced yes)
 		(effects
 			(font
@@
 	(label "ROW3"
 		(at 200.66 78.74 0)
-		(fields_autoplaced yes)
 		(effects
 			(font
@@
 	(label "ROW2"
 		(at 102.87 46.99 0)
-		(fields_autoplaced yes)
 		(effects
 			(font
@@
 	(label "COL1"
 		(at 58.42 31.75 0)
-		(fields_autoplaced yes)
 		(effects
 			(font
@@
 	(label "COL2"
 		(at 226.06 25.4 0)
-		(fields_autoplaced yes)
 		(effects
 			(font
@@
 	(label "COL2"
 		(at 58.42 35.56 0)
-		(fields_autoplaced yes)
 		(effects
 			(font
@@
 	(label "SDA"
 		(at 58.42 46.99 0)
-		(fields_autoplaced yes)
 		(effects
 			(font
@@
 	(label "COL3"
 		(at 243.84 25.4 0)
-		(fields_autoplaced yes)
 		(effects
 			(font
@@
 	(label "ROW3"
 		(at 102.87 50.8 0)
-		(fields_autoplaced yes)
 		(effects
 			(font
@@
 			)
 		)
-		(property "Footprint" "OPL:XIAO-RP2040-DIP"
+		(property "Footprint" "Module:MOUDLE14P-XIAO-DIP-SMD"
 			(at 83.058 58.928 0)
 			(effects
@@
 		)
 	)
+	(embedded_fonts no)
 )
